File: ecad/Crazyradio.sch (KiCad schematic (older format))
At the start: 36 parts, among them P1 USB-A-MALE, P2 CONN_5X2, U1 LP2985-33, U2 M74VHC1GT50, U3 NRF24LU1+, X1 CRYSTAL_SMD, Y1 CONREVSMA

Commit message: Rewrite using newer kicad and 0603 packages
Signed-off-by: Ziqian SUN(Zamir) <zsun@redhat.com>
Parts:
- removed D1, D2: DIODESCH, symbol DIODESCH
- removed P1: USB-A-MALE, symbol USB-A-MALE
- removed U1: LP2985-33, symbol LP2985-33
- removed U2: M74VHC1GT50, symbol MC74VHC1GT50
- removed X1: CRYSTAL_SMD, symbol CRYSTAL_SMD
- removed Y1: CONREVSMA, symbol CONREVSMA
- added AE1: Antenna_Chip, RF_Antenna:Texas_SWRA117D_2.4GHz_Right, symbol Device:Antenna_Chip
- added J1: USB_A, Icenowy_Connectors:USB_A, symbol Connector:USB_A
- added R10: 0R, Resistor_SMD:R_0603_1608Metric_Pad0.98x0.95mm_HandSolder, symbol Device:R_Small
- added U1: LP2985-3.3, Package_TO_SOT_SMD:SOT-23-5, symbol Regulator_Linear:LP2985-3.3
- added U2: SN74LV1T34DBV/74VHC1GT50, Package_TO_SOT_SMD:SOT-23-5, symbol Logic_LevelTranslator:SN74LV1T34DBV
- added Y2: Crystal_GND24, Crystal:Crystal_SMD_2520-4Pin_2.5x2.0mm, symbol Device:Crystal_GND24
- C1, C10, C11, C12, C13, C2, C3, C4, C5, C6, C7, C8, C9: footprint (none) -> Capacitor_SMD:C_0603_1608Metric_Pad1.08x0.95mm_HandSolder; symbol C -> Device:C_Small
- D3, D4: footprint (none) -> LED_SMD:LED_0603_1608Metric_Pad1.05x0.95mm_HandSolder; symbol LED -> Device:LED
- L1, L2, L3: footprint (none) -> Inductor_SMD:L_0603_1608Metric_Pad1.05x0.95mm_HandSolder; symbol INDUCTOR -> Device:L
- P2: footprint (none) -> Connector_PinHeader_2.54mm:PinHeader_2x05_P2.54mm_Vertical; symbol CONN_5X2 -> Connector_Generic:Conn_02x05_Odd_Even
- R1, R2, R3, R4, R5, R6, R7, R8, R9: footprint (none) -> Resistor_SMD:R_0603_1608Metric_Pad0.98x0.95mm_HandSolder; symbol R -> Device:R_Small
- U3: footprint (none) -> Package_DFN_QFN:QFN-32-1EP_5x5mm_P0.5mm_EP3.3x3.3mm; symbol NRF24LU1+ -> Crazyradio-rescue:NRF24LU1+
Connections:
- net labels added: +3V3
- net labels removed: 3V3
- wire segments 168 -> 150
